File: hardware/schematics/Laser Controller.kicad_sch (KiCad schematic)
At the start: 52 parts, among them J1 Micro_SD_Card, U1 ESP32-S3-N16R8-DevKit, U10 DS18B20, U12 OPA4134UA_2K5, U13 Galvo Input, U15 6N137, U16 6N137, U17 6N137, U2 DAC8562SDGST, U3 TTL_RGB Blue, U4 TTL_RGB Red, U5 TTL_RGB Green, U6 DS18B20, U7 DS18B20, U8 DS18B20, U9 DS18B20

Commit message: hw: op-amps finally got the memo about feedback
The galvo drive stage was running open-loop - OUT_A/OUT_B went straight to the
connector and nothing came back to the summing node, so the documented
Vout = 2.2 x (2.5V - Vdac) transfer simply did not exist in copper. Fixed the
X/Y channels, woke up the sleeping VREF buffer, and gave the supplies actual
sources instead of good intentions.

- R12/R17 (22k) moved from VREF to OUT_A/OUT_B -> both amps now close the loop
- R8 marked DNP; it skewed the summing node's DC operating point
- U12 unit C was a follower whose output fed nobody: R10/R15 now hang on
  OUT_C (VREF_BUF) instead of loading the DAC's VREFIN/OUT pin directly
- +15V rail had been merged onto the 5V opto supply (6N137 Vcc max is 7V) and
  -15V was a single dangling node - rails split, J2/J3 supply inlets added
- DAC8562 AVDD was unpowered; AVDD + CLR pull-up moved to +3V3 (it talks SPI
  to a 3V3 master), C1 returns to AGND
- C8 repurposed as U12 V+ decoupling, unused unit D's +IN tied to AGND
- SD socket ground reached the MCU module only, never the board ground net
- R26 / U3 / U4 / U5 got the footprints they were missing
- R27-R29: the 10k fail-safe pull-ups on GPIO7/8/21 that keep the laser OFF
  at boot and on crash - documented as pending, now in the schematic
- PWR_FLAGs on every rail: ERC 11 errors -> 1 (SD CLK pin is typed
  "power input" in KiCad's own Micro_SD_Card symbol)
Parts:
- added J2: PWR IN +5V, Connector_PinHeader_2.54mm:PinHeader_1x02_P2.54mm_Vertical, symbol Connector:Conn_01x02_Socket
- added J3: PWR IN Galvo, Connector_PinHeader_2.54mm:PinHeader_1x04_P2.54mm_Vertical, symbol Connector:Conn_01x04_Socket
- added R27, R28, R29: 10k, Resistor_THT:R_Axial_DIN0204_L3.6mm_D1.6mm_P1.90mm_Vertical, symbol Device:R
- R26: footprint (none) -> Resistor_THT:R_Axial_DIN0204_L3.6mm_D1.6mm_P1.90mm_Vertical
- R8: now not fitted
- U3, U4, U5: footprint (none) -> Connector_PinHeader_2.54mm:PinHeader_1x02_P2.54mm_Vertical
Connections:
- net +15V: now also C8.1, J3.1 (Pin_1); no longer C5.1, C6.1, C7.1, D1.2 (A), U15.7 (EN), U15.8 (VCC), U16.7 (EN), U16.8 (VCC), U17.7 (EN), U17.8 (VCC)
- net -15V: now also J3.4 (Pin_4)
- net 5V GND Buck: now also J1.6 (GND), U1.J2_1 (GND), J2.2 (Pin_2)
- net AGND (from Galvo Board): now also C1.2, C8.2, U12.12 (+IN_D), J3.2 (Pin_2), J3.3 (Pin_3)
- net Buck +5V: now also C5.1, C6.1, C7.1, D1.2 (A), U15.7 (EN), U15.8 (VCC), U16.7 (EN), U16.8 (VCC), U17.7 (EN), U17.8 (VCC), J2.1 (Pin_1)
- net +3V3: now reaches J1.1 (3v3), R18.1, R20.1, R22.1, R5.2, U1.J1_1 (3V3), U1.J1_2 (3V3), U10.3 (V_{DD}), U6.3 (V_{DD}), U7.3 (V_{DD}), U8.3 (V_{DD}), U9.3 (V_{DD})
- net +3V3: now also C1.1, R3.2, U2.9 (AVDD), R27.1, R28.1, R29.1
- net VREF_BUF: now reaches U12.8 (OUT_C), U12.9 (-IN_C)
- net VREF_BUF: now also R10.2, R15.2; no longer C8.1
- net at R16.1, U12.7 (OUT_B): now also R17.2
- net +5V_MCU: now reaches D1.1 (K), U1.J1_21 (5V0)
- net +5V_MCU: no longer C1.2, R3.2
- net at R6.1, U12.1 (OUT_A): now also R12.1
- net GPIO21: now reaches R4.1, U1.J2_18 (GPIO21)
- net GPIO21: now also R29.2
- net GPIO8: now reaches R2.1, U1.J1_12 (GPIO8)
- net GPIO8: now also R28.2
- net GPIO7: now reaches R1.1, U1.J1_7 (GPIO7)
- net GPIO7: now also R27.2
- new net: C2.1, U12.10 (+IN_C), U2.10 (VREFINNREFOUT)
- no-connect marks 34 -> 33
Other:
- note added: "FAIL-SAFE PULL-UPS - laser OFF on boot/crash"
- note added: "RAIL FLAGS (ERC)"
- note added: "SUPPLY INLETS"
- moved on the sheet: C8

Commit message: hw: everything's JST XH now, the fans finally get a seat at the table
RGB, DS18B20 probes, +5V/+-15V supply and the galvo signal input all
standardized onto JST XH 2.54mm housings -- J3 and U13 lost a stray
unused pin in the process (4-pin -> clean 3-pin). Two fan sub-circuits
added from scratch (J4-J7, R30/R31): 2-pin JST power feed -> standard
4-pin PC-fan header, PWM straight off GPIO16/17 (no driver stage --
that's what a real 4-wire fan's PWM pin is for), TACH wired to the two
GPIOs that have been sitting free since the SD rewire (2 and 9),
hardware-only for now.

Board was full at 118x90, stretched to 118x115 for the new fan row.
Freerouting 2.2.4 did a full re-route (footprint swaps orphaned most
of the old copper), zones refilled, DRC down to 4 pre-existing
zone-corner nitpicks that have nothing to do with any of this.
Parts:
- removed J3: PWR IN Galvo, Connector_PinHeader_2.54mm:PinHeader_1x04_P2.54mm_Vertical, symbol Connector:Conn_01x04_Socket
- removed U13: Galvo Input, Connector_FFC-FPC:TE_84982-4_2Rows-04Pins-P1.0mm_Vertical, symbol Connector:Conn_01x04_Socket
- added J3: PWR IN Galvo, Connector_JST:JST_XH_B3B-XH-A_1x03_P2.50mm_Vertical, symbol Connector:Conn_01x03_Socket
- added J4: FAN1 PWR IN, Connector_JST:JST_XH_B2B-XH-A_1x02_P2.50mm_Vertical, symbol Connector:Conn_01x02_Socket
- added J5: FAN1, Connector_PinHeader_2.54mm:PinHeader_1x04_P2.54mm_Vertical, symbol Connector:Conn_01x04_Socket
- added J6: FAN2 PWR IN, Connector_JST:JST_XH_B2B-XH-A_1x02_P2.50mm_Vertical, symbol Connector:Conn_01x02_Socket
- added J7: FAN2, Connector_PinHeader_2.54mm:PinHeader_1x04_P2.54mm_Vertical, symbol Connector:Conn_01x04_Socket
- added R30, R31: 4.7k, Resistor_THT:R_Axial_DIN0204_L3.6mm_D1.6mm_P1.90mm_Vertical, symbol Device:R
- added U13: Galvo Input, Connector_JST:JST_XH_B3B-XH-A_1x03_P2.50mm_Vertical, symbol Connector:Conn_01x03_Socket
- J2, U3, U4, U5: footprint Connector_PinHeader_2.54mm:PinHeader_1x02_P2.54mm_Vertical -> Connector_JST:JST_XH_B2B-XH-A_1x02_P2.50mm_Vertical
- U10, U6, U7, U8, U9: footprint Package_TO_SOT_THT:TO-92_Inline -> Connector_JST:JST_XH_B3B-XH-A_1x03_P2.50mm_Vertical
Connections:
- net +15V: now also J3.1 (Pin_1); no longer C8.1
- net +3V3: now also R30.1, R31.1
- net -15V: now also J3.3 (Pin_3)
- net 5V GND Buck: now also J4.2 (Pin_2), J5.1 (Pin_1), J6.2 (Pin_2), J7.1 (Pin_1)
- net AGND (from Galvo Board): now also J3.2 (Pin_2), U13.1 (Pin_1)
- net Buck +5V: now also J4.1 (Pin_1), J5.2 (Pin_2), J6.1 (Pin_1), J7.2 (Pin_2); no longer C5.1, C6.1, C7.1, D1.2 (A), U15.7 (EN), U15.8 (VCC), U16.7 (EN), U16.8 (VCC), U17.7 (EN), U17.8 (VCC)
- net at R16.1, U12.7 (OUT_B): no longer R17.2
- net at R16.2: now also U13.3 (Pin_3)
- net at C2.1, U2.10 (VREFINNREFOUT): no longer U12.10 (+IN_C)
- net at R6.1, U12.1 (OUT_A): no longer R12.1
- net at R6.2: now also U13.2 (Pin_2)
- net FAN2_PWM: now reaches U1.J1_10 (GPIO17)
- net FAN2_PWM: now also J7.4 (Pin_4)
- net FAN1_TACH: now reaches U1.J1_15 (GPIO9)
- net FAN1_TACH: now also J5.3 (Pin_3), R30.2
- net FAN1_PWM: now reaches U1.J1_9 (GPIO16)
- net FAN1_PWM: now also J5.4 (Pin_4)
- net FAN2_TACH: now reaches U1.J2_5 (GPIO2)
- net FAN2_TACH: now also J7.3 (Pin_3), R31.2
- new net: C5.1, C6.1, C7.1, D1.2 (A), U15.7 (EN), U15.8 (VCC), U16.7 (EN), U16.8 (VCC), U17.7 (EN), U17.8 (VCC)
- no-connect marks 33 -> 28

Commit message: hw: KiCad project catches up on ERC bookkeeping / docs: a caption goes on a diet
Schematic/PCB/project files re-saved after running ERC in KiCad -- pin_map,
erc_exclusions and per-sheet instance data now live in the .kicad_pro, and
the newer format's extra per-symbol fields (do_not_autoplace, show_name,
etc.) landed in the .kicad_sch/.kicad_pcb along the way. No intentional
routing/placement changes.

docs/01-introduction.md's prototype-board photo caption gets trimmed; the
/update page's Chapter 3 walkthrough drops a now-redundant screenshot note.
Parts:
- removed R8: 22k, Resistor_THT:R_Axial_DIN0204_L3.6mm_D1.6mm_P1.90mm_Vertical, symbol Device:R
Connections:
- net at R6.1, U12.1 (OUT_A): now also R12.1
Other:
- moved on the sheet: J4, J5, R30, R31, R6, R7

Commit message: Add files via upload
Other:
- title: ESP32 Laser Controller Board -> GalvOS ESP32 Laser Controller Board
Changed lines of the file:
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@@
 	(paper "A2")
 	(title_block
-		(title "ESP32 Laser Controller Board")
+		(title "GalvOS ESP32 Laser Controller Board")
 		(date "2026-07-24")
 	)

Commit message: Add files via upload
Other:
- title: GalvOS ESP32 Laser Controller Board -> GalvOS ESP32 Laser Controller Board V1.2.0
Changed lines of the file:
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@@
 	(paper "A2")
 	(title_block
-		(title "GalvOS ESP32 Laser Controller Board")
+		(title "GalvOS ESP32 Laser Controller Board V1.2.0")
 		(date "2026-07-24")
 	)

Commit message: Add files via upload
Other:
- title: GalvOS ESP32 Laser Controller Board V1.2.0 -> GalvOS ESP32 Laser Controller Board V1.2.1
Changed lines of the file:
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@@
 	(paper "A2")
 	(title_block
-		(title "GalvOS ESP32 Laser Controller Board V1.2.0")
+		(title "GalvOS ESP32 Laser Controller Board V1.2.1")
 		(date "2026-07-24")
 	)

Commit message: Add files via upload
Other:
- title: GalvOS ESP32 Laser Controller Board V1.2.1 -> GalvOS ESP32 Laser Controller Board V1.2.2
Changed lines of the file:
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@@
 	(paper "A2")
 	(title_block
-		(title "GalvOS ESP32 Laser Controller Board V1.2.1")
+		(title "GalvOS ESP32 Laser Controller Board V1.2.2")
 		(date "2026-07-24")
 	)

Commit message: Add files via upload
Other:
- title: GalvOS ESP32 Laser Controller Board V1.2.2 -> GalvOS ESP32 Laser Controller Board V1.2.3
Changed lines of the file:
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@@
 	(paper "A2")
 	(title_block
-		(title "GalvOS ESP32 Laser Controller Board V1.2.2")
+		(title "GalvOS ESP32 Laser Controller Board V1.2.3")
 		(date "2026-07-24")
 	)
