File: hardware/schematics/Laser Controller.kicad_sch (KiCad schematic)
At the start: 62 parts, among them J1 Micro_SD_Card, J2 PWR IN +5V, J3 PWR IN Galvo, J4 FAN1 PWR IN, J5 FAN1, J6 FAN2 PWR IN, J7 FAN2, U1 ESP32-S3-N16R8-DevKit, U10 DS18B20, U12 OPA4134UA_2K5, U13 Galvo Input, U15 6N137, U16 6N137, U17 6N137, U2 DAC8562SDGST, U3 TTL_RGB Blue, U4 TTL_RGB Red, U5 TTL_RGB Green, U6 DS18B20, U7 DS18B20, U8 DS18B20, U9 DS18B20

Commit message: Add files via upload
Other:
- title: GalvOS ESP32 Laser Controller Board V1.2.3 -> GalvOS ESP32 Laser Controller Board V1.2.4
Changed lines of the file:
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@@
 	(paper "A2")
 	(title_block
-		(title "GalvOS ESP32 Laser Controller Board V1.2.3")
+		(title "GalvOS ESP32 Laser Controller Board V1.2.4")
 		(date "2026-07-24")
 	)

Commit message: Add files via upload
Other:
- title: GalvOS ESP32 Laser Controller Board V1.2.4 -> GalvOS ESP32 Laser Controller Board V1.2.5
Changed lines of the file:
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@@
 	(paper "A2")
 	(title_block
-		(title "GalvOS ESP32 Laser Controller Board V1.2.4")
+		(title "GalvOS ESP32 Laser Controller Board V1.2.5")
 		(date "2026-07-24")
 	)

Commit message: Add files via upload
Other:
- title: GalvOS ESP32 Laser Controller Board V1.2.5 -> GalvOS ESP32 Laser Controller Board V1.2.6
Changed lines of the file:
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@@
 	(paper "A2")
 	(title_block
-		(title "GalvOS ESP32 Laser Controller Board V1.2.5")
+		(title "GalvOS ESP32 Laser Controller Board V1.2.6")
 		(date "2026-07-24")
 	)

Commit message: test kibot
Other:
- title: GalvOS ESP32 Laser Controller Board V1.2.6 -> GalvOS ESP32 Laser Controller Board V1.2.7
Changed lines of the file:
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@@
 	(paper "A2")
 	(title_block
-		(title "GalvOS ESP32 Laser Controller Board V1.2.6")
+		(title "GalvOS ESP32 Laser Controller Board V1.2.7")
 		(date "2026-07-24")
 	)

Commit message: Update .gitignore and add branch-meta.json for token saving
Parts:
- J5, J7: footprint Connector_PinHeader_2.54mm:PinHeader_1x04_P2.54mm_Vertical -> Connector_Molex:Molex_KK-254_AE-6410-04A_1x04_P2.54mm_Vertical
Changed lines of the file:
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@@
 			)
 		)
-		(property "Footprint" "Connector_PinHeader_2.54mm:PinHeader_1x04_P2.54mm_Vertical"
+		(property "Footprint" "Connector_Molex:Molex_KK-254_AE-6410-04A_1x04_P2.54mm_Vertical"
 			(at 464.82 100.33 0)
 			(hide yes)
@@
 			)
 		)
-		(property "Footprint" "Connector_PinHeader_2.54mm:PinHeader_1x04_P2.54mm_Vertical"
+		(property "Footprint" "Connector_Molex:Molex_KK-254_AE-6410-04A_1x04_P2.54mm_Vertical"
 			(at 468.63 134.62 0)
 			(hide yes)

Commit message: hw: v6.85.0 -- swap DS18B20/RGB/J3 to real JST-XH footprints, not just relabeled ones
- U6-U10 (DS18B20): were still physically the old TO-92 sensor pads
  wearing a JST-XH label (descr/tags still said TO-92). Delete+resync
  from schematic + reposition + reroute -> genuine
  JST_XH_B3B-XH-A_1x03_P2.50mm_Vertical, verified against library.
- U3-U5 (RGB TTL): same bug, same fix -> genuine
  JST_XH_B2B-XH-A_1x02_P2.50mm_Vertical.
- Gave the DS18B20 1-Wire bus an explicit net label (was unnamed,
  which is why pads kept losing their net assignment mid-swap).
- Rewired the 1-Wire + 3V3 daisy chain across all 5 sensors to the
  new pad positions without touching the working legacy trunk.
- J3 (PWR IN Galvo): finished the 3-pin -> 4-pin JST-XH swap properly
  (schematic symbol + footprint), pin 4 wired to -15V.
- ESP32 socket: confirmed the existing devkit footprint IS already a
  proper 2x22 2.54mm THT pin-socket pattern -- added silkscreen note
  + BOM property instead of a needless footprint swap.

Known follow-up: J_DMX and U13 have the same label-only-fix bug,
not yet corrected. DS18B20 column spacing (9mm) is tighter than a
real JST-XH B3B housing needs (~11mm) -- courtyards overlap by
~2x6.8mm, electrically harmless but a real assembly fit issue.

Zero shorts, zero solder-mask bridges, zero missing-net pads on the
touched components; lib_footprint_mismatch confirms U3-U10 now match
the real library parts.
Parts:
- removed J1: Micro_SD_Card, Connector_Card:SD_Card_Device_16mm_SlotDepth, symbol Connector:Micro_SD_Card
- removed J3: PWR IN Galvo, Connector_JST:JST_XH_B3B-XH-A_1x03_P2.50mm_Vertical, symbol Connector:Conn_01x03_Socket
- added C_ANA1: 10uF, Capacitor_SMD:C_0805_2012Metric, symbol Device:C
- added C_ANA2, C_BOOT, C_INHF, C_SCANX, C_SCANY, C_WD1: 100nF, Capacitor_SMD:C_1206_3216Metric, symbol Device:C
- added C_IN1, C_IN2: 10uF, Capacitor_SMD:C_1210_3225Metric, symbol Device:C
- added C_OUT1, C_OUT2: 22uF, Capacitor_SMD:C_1210_3225Metric, symbol Device:C
- added C_SCANCONT, C_SCANT, C_WDCONT: 10nF, Capacitor_SMD:C_1206_3216Metric, symbol Device:C
- added C_TRIGC_WD: 1nF, Capacitor_SMD:C_1206_3216Metric, symbol Device:C
- added C_VCC: 1uF, Capacitor_SMD:C_1206_3216Metric, symbol Device:C
- added D2: 1N5822, Diode_THT:D_DO-201AD_P15.24mm_Horizontal, symbol Diode:1N5822
- added D_TRIGCL_SCAN, D_TRIGCL_WD: 1N4148, Diode_SMD:D_SOD-123, symbol Diode:1N4148
- added FB1: BLM18PG221SN1, Inductor_SMD:L_0603_1608Metric, symbol Device:FerriteBead_Small
- added J1: SD Card Module (6-pin, 2.54mm), Connector_PinSocket_2.54mm:PinSocket_1x06_P2.54mm_Vertical, symbol Connector:Conn_01x06_Socket
- added J3: PWR IN Galvo, Connector_JST:JST_XH_B4B-XH-A_1x04_P2.50mm_Vertical, symbol Connector:Conn_01x04_Socket
- added J_DMX: DMX MAX485, Connector_PinSocket_2.54mm:PinSocket_1x04_P2.54mm_Vertical, symbol Connector:Conn_01x04_Socket
- added J_ESTOP: E-STOP, Connector_JST:JST_XH_B2B-XH-A_1x02_P2.50mm_Vertical, symbol Connector:Conn_01x02_Socket
- added J_SSR1: SSR1 CTRL, Connector_JST:JST_XH_B2B-XH-A_1x02_P2.50mm_Vertical, symbol Connector:Conn_01x02_Socket
- added L1: 6.8uH, Inductor_SMD:L_Sunlord_MWSA1204S-6R8, symbol Device:L
- added R_EN1: 63.4k 1%, Resistor_SMD:R_1206_3216Metric, symbol Device:R
- added R_EN2: 10k 1%, Resistor_SMD:R_1206_3216Metric, symbol Device:R
- added R_FB1: 100k 1%, Resistor_SMD:R_1206_3216Metric, symbol Device:R
- added R_FB2: 24.9k 1%, Resistor_SMD:R_1206_3216Metric, symbol Device:R
- added R_SCANT: 1.8M, Resistor_SMD:R_1206_3216Metric, symbol Device:R
- added R_SSRCTRL: 330, Resistor_SMD:R_1206_3216Metric, symbol Device:R
- added R_TRIGPU_SCAN, R_TRIGPU_WD: 10k, Resistor_SMD:R_1206_3216Metric, symbol Device:R
- added R_WD1: 910k 1%, Resistor_SMD:R_1206_3216Metric, symbol Device:R
- added U_BUCK: LMR33630ADDA, Package_SO:Texas_HSOP-8-1EP_3.9x4.9mm_P1.27mm_ThermalVias, symbol Regulator_Switching:LMR33630ADDA
- added U_SCAN, U_WD: NE555D, Package_SO:SOIC-8_3.9x4.9mm_P1.27mm, symbol Timer:NE555D
- J2: value PWR IN +5V -> PWR IN VIN_BUCK (10-30V)
- U1: Assembly (none) -> Mounted via 2x 1x22 2.54mm female pin socket strip (footpri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
Connections:
- net +15V: now also J3.1 (Pin_1)
- net +3V3: now also J1.1 (Pin_1); no longer C1.1, U2.9 (AVDD)
- net -15V: now also R14.2, Y_Knoten1.2, C_SCANX.1, C_SCANY.1, C_SCANY.2, D_TRIGCL_SCAN.1 (K), J3.3 (Pin_3), J3.4 (Pin_4), R_TRIGPU_SCAN.2, U_SCAN.2 (TRIG)
- net 5V GND Buck: now also C_IN1.2, C_IN2.2, C_INHF.2, C_OUT1.2, C_OUT2.2, C_SCANCONT.2, C_SCANT.2, C_VCC.2, C_WD1.2, C_WDCONT.2, D_TRIGCL_SCAN.2 (A), D_TRIGCL_WD.2 (A), J1.6 (Pin_6), J_DMX.2 (Pin_2), J_ESTOP.2 (Pin_2), J_SSR1.2 (Pin_2), R_EN2.2, R_FB2.2, U_BUCK.1 (GND), U_BUCK.9 (GND), U_SCAN.1 (GND), U_WD.1 (GND)
- net AGND (from Galvo Board): now also C_ANA1.2, C_ANA2.2, J3.2 (Pin_2)
- net Buck +5V: now also C_OUT1.1, C_OUT2.1, FB1.1, J_DMX.1 (Pin_1), L1.2, R_FB1.1, R_SCANT.1, R_TRIGPU_SCAN.1, R_TRIGPU_WD.1, R_WD1.1, U_SCAN.4 (~{RST}), U_SCAN.8 (VCC), U_WD.8 (VCC); no longer J2.1 (Pin_1)
- net at R7.2, X_Knoten1.2: now also C_SCANX.2
- net DS18B20_1WIRE: now reaches R5.1, U1.J1_11 (GPIO18), U10.2 (DQ), U6.2 (DQ), U7.2 (DQ), U8.2 (DQ), U9.2 (DQ)
- net TTL_RGB_GREEN: now reaches R20.2, R21.1, U16.6 (VO), U5.2 (Pin_2)
- net TTL_RGB_RED: now reaches R18.2, R19.1, U15.6 (VO), U4.2 (Pin_2)
- net SD_CS: now reaches U1.J2_6 (GPIO42)
- net SD_CS: now also J1.2 (Pin_2)
- net SD_MOSI: now reaches U1.J1_6 (GPIO6)
- net SD_MOSI: now also J1.3 (Pin_3)
- net SD_SCK: now reaches U1.J1_5 (GPIO5)
- net SD_SCK: now also J1.4 (Pin_4)
- net SD_MISO: now reaches U1.J2_4 (GPIO1)
- net SD_MISO: now also J1.5 (Pin_5)
- net GPIO14: now reaches U1.J1_20 (GPIO14)
- net GPIO14: now also C_TRIGC_WD.1
- net GPIO4: now reaches U1.J1_4 (GPIO4)
- net GPIO4: now also J_DMX.3 (Pin_3)
- net GPIO38: now reaches U1.J2_10 (GPIO38)
- net GPIO38: now also U_WD.4 (~{RST})
- net GPIO47: now reaches U1.J2_17 (GPIO47)
- net GPIO47: now also J_ESTOP.1 (Pin_1)
- net GPIO39: now reaches U1.J2_9 (GPIO39)
- net GPIO39: now also U_SCAN.3 (OUT)
- net TTL_RGB_BLUE: now reaches R22.2, R23.1, U17.6 (VO), U3.2 (Pin_2)
- new net +5V_ANA: C1.1, C_ANA1.1, C_ANA2.1, FB1.2, U2.9 (AVDD)
- new net BOOT_BUCK: C_BOOT.2, U_BUCK.7 (BOOT)
- new net EN_BUCK: R_EN1.2, R_EN2.1, U_BUCK.3 (EN)
- new net FB_BUCK: R_FB1.2, R_FB2.1, U_BUCK.5 (FB)
- new net SCAN_CONT: C_SCANCONT.1, U_SCAN.5 (CONT)
- new net SCAN_RC: C_SCANT.1, R_SCANT.2, U_SCAN.6 (THRES), U_SCAN.7 (DISCH)
- new net SSR1_CTRL: J_SSR1.1 (Pin_1), R_SSRCTRL.2
- new net SW_BUCK: C_BOOT.1, L1.1, U_BUCK.8 (SW)
- new net VCC_BUCK: C_VCC.1, U_BUCK.6 (VCC)
- new net VIN_BUCK: C_IN1.1, C_IN2.1, C_INHF.1, D2.1 (K), R_EN1.1, U_BUCK.2 (VIN)
- new net VIN_RAW: D2.2 (A), J2.1 (Pin_1)
- new net WD_CONT: C_WDCONT.1, U_WD.5 (CONT)
- new net WD_OUT: R_SSRCTRL.1, U_WD.3 (OUT)
- new net WD_RC: C_WD1.1, R_WD1.2, U_WD.6 (THRES), U_WD.7 (DISCH)
- new net WD_TRIG: C_TRIGC_WD.2, D_TRIGCL_WD.1 (K), R_TRIGPU_WD.2, U_WD.2 (TRIG)
- no-connect marks 28 -> 25

Commit message: hw: v6.86.0 -- J3 and J_DMX finally get real JST-XH bodies, DS18B20 quintet marches into a single file
- J3 (PWR IN Galvo) and J_DMX: swapped the leftover PinSocket-shaped copper
  for the actual JST_XH_B4B-XH-A_1x04 pads/courtyard/silk (previous pass only
  renamed the footprint field, geometry never followed). Repositioned/rotated
  to match, all nets re-verified pad-for-pad against the old routing.
- U6-U10 (DS18B20): the two-column layout put real B3B-XH-A housings only
  9mm apart (need ~11mm not to collide) -- courtyards overlapped by ~2x6.8mm.
  Collapsed all five into one vertical column with >=9mm pitch (one wider
  gap to dodge R31), rebuilt the DS18B20_1WIRE and +3V3 local bus wiring
  (two vias added to hop the existing +3V3 trunk crossing) to match.
- Verified: check_courtyard_overlaps clean for all six connectors, no new
  shorts/crossings introduced (DRC-diffed against baseline).

Known follow-up (not touched this round, needs a call):
- U13 (Galvo Input) footprint field says JST_XH_B3B-XH-A_1x03 but the
  placed copper is 4 SMD pads that don't match a 3-pin THT JST at all --
  worse than the J3/J_DMX bug, needs the real part identified first.
- J2 (PWR IN +5V) has the exact same label-only bug J3 had: JST_XH_B2B-XH-A
  in the footprint field, old PinSocket-shaped copper underneath.
- Zone refill needed in KiCad (Edit > Fill Zones, hotkey B) -- the GND pour
  wasn't recomputed around the new copper, so DRC still shows stale
  zone-clearance/solder-mask-bridge noise at the new pad/via spots until
  that runs. MCP's own refill_zones has a known segfault risk on this
  backend, so left it for the UI.
- Pre-existing +3V3/FAN1_PWM clearance nits near U3 and the top-left
  starved-thermal/silk warnings untouched, as requested.
Parts:
- J_DMX: footprint Connector_PinSocket_2.54mm:PinSocket_1x04_P2.54mm_Vertical -> Connector_JST:JST_XH_B4B-XH-A_1x04_P2.50mm_Vertical
Changed lines of the file:
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@@
 			)
 		)
-		(property "Footprint" "Connector_PinSocket_2.54mm:PinSocket_1x04_P2.54mm_Vertical"
+		(property "Footprint" "Connector_JST:JST_XH_B4B-XH-A_1x04_P2.50mm_Vertical"
 			(at 110.49 400.05 0)
 			(hide yes)
