File: hardware/schematics/Laser Controller.kicad_sch (KiCad schematic)
At the start: 98 parts, among them J1 SD Card Module (6-pin, 2.54mm), J2 PWR IN VIN_BUCK (10-30V), J3 PWR IN Galvo, J4 FAN1 PWR IN, J5 FAN1, J6 FAN2 PWR IN, J7 FAN2, U1 ESP32-S3-N16R8-DevKit, U10 DS18B20, U12 OPA4134UA_2K5, U13 Galvo Input, U15 6N137, U16 6N137, U17 6N137, U2 DAC8562SDGST, U3 TTL_RGB Blue, U4 TTL_RGB Red, U5 TTL_RGB Green, U6 DS18B20, U7 DS18B20, U8 DS18B20, U9 DS18B20

Commit message: hw: v6.88.0 -- the axial resistors trade their leads for landing pads
Swapped 32 THT axial resistors (all the 1k/10k/22k pull-ups, dividers,
and 0-ohm jumpers) plus 8 miswired-footprint decoupling caps from
CP_Radial to real Capacitor_SMD, all onto 1206 SMD to match the rest
of the board's existing SMD convention. Buck output caps C_OUT1/2
downsized 1210->1206 (5V rail, plenty of voltage margin).

Left alone on purpose: C_IN1/C_IN2 stay 1210 (10-30V input needs a
voltage rating 1206 can't reliably deliver at 10uF), L1 stays a real
shielded power inductor (no chip inductor eats buck-converter amps),
FB1 stays 0603 (already smaller than asked for).

Routing is now stale -- pad positions moved, so this needs a
re-place + re-route pass in KiCad before it's fab-ready.
Parts:
- C1, C2, C3, C4, C5, C6, C7, C8: footprint Capacitor_THT:CP_Radial_D4.0mm_P1.50mm -> Capacitor_SMD:C_1206_3216Metric
- C_OUT1, C_OUT2: footprint Capacitor_SMD:C_1210_3225Metric -> Capacitor_SMD:C_1206_3216Metric
- R1, R10, R11, R12, R13, R14, R15, R16, R17, R18, R19, R2, R20, R21, R22, R23, R25, R26, R27, R28, R29, R3, R30, R31, R4, R5, R6, R7, R9, X_Knoten1, Y_Knoten1: footprint Resistor_THT:R_Axial_DIN0204_L3.6mm_D1.6mm_P1.90mm_Vertical -> Resistor_SMD:R_1206_3216Metric
Connections:
- net -15V: no longer R14.2, Y_Knoten1.2
- net DS18B20_1WIRE: no longer names the net of R5.1, U1.J1_11 (GPIO18), U10.2 (DQ), U6.2 (DQ), U7.2 (DQ), U8.2 (DQ), U9.2 (DQ)
- new net: R14.2, Y_Knoten1.2
Other:
- moved on the sheet: C_BOOT, C_OUT1, C_OUT2, J4, J5, J6, J7, L1, R_FB1, R_FB2
