File: hardware/schematics/Laser Controller.kicad_sch (KiCad schematic)
At the start: 98 parts, among them J1 SD Card Module (6-pin, 2.54mm), J2 PWR IN VIN_BUCK (10-30V), J3 PWR IN Galvo, J4 FAN1 PWR IN, J5 FAN1, J6 FAN2 PWR IN, J7 FAN2, U1 ESP32-S3-N16R8-DevKit, U10 DS18B20, U12 OPA4134UA_2K5, U13 Galvo Input, U15 6N137, U16 6N137, U17 6N137, U2 DAC8562SDGST, U3 TTL_RGB Blue, U4 TTL_RGB Red, U5 TTL_RGB Green, U6 DS18B20, U7 DS18B20, U8 DS18B20, U9 DS18B20

Commit message: hw: Laser Controller schematic gets a haircut, netlist keeps its DNA
Layout and hygiene pass on the single-sheet Laser Controller schematic.
Every edit was netlist-verified: kicad-cli netlist export before/after,
92 nets on both sides, exactly one intentional electrical change.

Electrical (the only one):
- C_SCANY sat directly on the -15V rail, its "connecting" wire started at
  the symbol origin instead of a pin. It now sits on the Y_NODE1 damping
  node where it belongs, mirroring C_SCANX on the X channel.

Layout:
- RGB TTL divider block re-spaced: R18/R19 no longer touch pin-to-pin,
  they get the same 2.54 mm gap as R22/R23. GREEN feed rerouted around
  R19's new body with a jog at x=412.75.
- R21 pulled down onto the GND rail endpoint, #PWR39 moved out of U1's
  bounding box.
- 18 wires crossing symbol bodies: now 0. Overlapping elements: 0.
  Orphaned wires: 0. Off-grid geometry: none.

References:
- X_Knoten1/Y_Knoten1 renamed to X_NODE1/Y_NODE1 (English only, per
  project convention).
- 20 designators without a trailing digit got one (C_BOOT -> C_BOOT1
  and friends). KiCad considered them un-annotated; that warning is gone.

Libraries:
- Project-scoped sym-lib-table and fp-lib-table added, pointing at
  KiCad_Libs. Symbol-pin to footprint-pad mapping verified 1:1 for
  U1 (44/44), U2 (10/10) and U12 (14/14).
- The ESP32-S3 DevKit symbol in KiCad_Libs is deliberately NOT registered:
  it is a 40-pin variant while the board uses the 44-pin DevKitC-1.
  Re-linking it would silently remap GPIO8/14/21 - laser G/B TTL and the
  watchdog heartbeat. Not the kind of surprise you want from a Class 4
  device. Needs a corrected symbol before it can be wired up.

ERC: 0 errors, 226 warnings - all of them "library not in current
configuration" from the stock KiCad libs not being installed on this
machine, plus one benign PWR_FLAG pin_to_pin note.

Co-Authored-By: Claude Opus 5 <noreply@anthropic.com>
Parts:
- renumbered C_BOOT to C_BOOT1, C_INHF to C_INHF1, C_SCANCONT to C_SCANCONT1, C_SCANT to C_SCANT1, C_SCANX to C_SCANX1, C_SCANY to C_SCANY1, C_TRIGC_WD to C_TRIGC_WD1, C_VCC to C_VCC1, C_WDCONT to C_WDCONT1, D_TRIGCL_SCAN to D_TRIGCL_SCAN1, D_TRIGCL_WD to D_TRIGCL_WD1, J_DMX to J_DMX1, J_ESTOP to J_ESTOP1, R_SCANT to R_SCANT1, R_SSRCTRL to R_SSRCTRL1, R_TRIGPU_SCAN to R_TRIGPU_SCAN1, R_TRIGPU_WD to R_TRIGPU_WD1, U_BUCK to U_BUCK1, U_SCAN to U_SCAN1, U_WD to U_WD1, X_Knoten1 to X_NODE1, Y_Knoten1 to Y_NODE1
Connections:
- net -15V: no longer C_SCANX1.1, C_SCANY1.1, C_SCANY1.2, D_TRIGCL_SCAN1.1 (K), R_TRIGPU_SCAN1.2, U_SCAN1.2 (TRIG)
- net at R14.2, Y_NODE1.2: now also C_SCANY1.2
- new net SCAN_TRIG: C_SCANX1.1, C_SCANY1.1, D_TRIGCL_SCAN1.1 (K), R_TRIGPU_SCAN1.2, U_SCAN1.2 (TRIG)
Other:
- note added: "+5V ANALOG SUPPLY FILTER"
- note added: "BUCK CONVERTER LMR33630 - VIN 10-30V TO +5V"
- note added: "DAC8562 - DUAL 16-BIT DAC (SPI2)"
- note added: "ESP32-S3-N16R8 CONTROLLER"
- note added: "EXTERNAL INTERFACES - E-STOP / DMX / SSR"
- note added: "FAN CONTROL + TACHO"
- note added: "GALVO ANALOG OUTPUT - OPA4134"
- note added: "HARDWARE WATCHDOG - NE555"
- note added: "LASER TTL ISOLATION - 6N137 (INVERTED)"
- note added: "SCAN-FAIL DETECTOR - NE555"
- note added: "SD CARD (SPI3)"
- note added: "TEMPERATURE SENSORS - DS18B20 1-WIRE"
- moved on the sheet: C_SCANX1, C_SCANY1, J1, R19, R21

Commit message: hw: ERC drops from 225 warnings to 1, symbol libraries finally show up
Installed kicad-library/kicad-library-3d, so every stock Device:R,
Device:C, power:*, Connector:* and friends now resolve instead of
shouting into the void.

Cleanup of what the newly-visible libraries exposed:

- ESP32-S3-N16R8-DevKit retargeted from the stock RF_Module nickname
  (which never had a DevKit symbol) to a new ESP32 entry in the project
  sym-lib-table pointing at the custom library.
- Regenerated that custom library FROM the schematic, not the other way
  around: the on-disk copy had 41 pins instead of 44 and its GPIO map
  slipped by one from J1_12 onward, which would have quietly moved
  Laser G off GPIO8 onto GPIO3. The schematic and the netlist agreed
  with the real DevKitC-1 header, so the file lost the argument.
- Refreshed the cached DS18B20, LMR33630ADDA and NE555D symbols from
  the stock libraries.
- Regenerated the netlist, which was stale: 75 nets before, 92 now.
  The fan PWM/tach lines, the buck's BOOT/EN/FB nets, GPIO4/38/39 and
  +5V_ANA had been missing.

Verified: canonical connectivity diff (net name to sorted ref.pin set)
before and after the symbol refresh is byte-identical. No pin moved,
no wire came loose.

Remaining ERC warning is a pre-existing design question, not a library
one: a PWR_FLAG shares a net with the DAC8562 LDAC pin.

Co-Authored-By: Claude Opus 5 <noreply@anthropic.com>
Parts:
- U1: symbol RF_Module:ESP32-S3-N16R8-DevKit -> ESP32:ESP32-S3-N16R8-DevKit
Changed lines of the file:
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@@
 	)
 	(symbol
-		(lib_id "RF_Module:ESP32-S3-N16R8-DevKit")
+		(lib_id "ESP32:ESP32-S3-N16R8-DevKit")
 		(at 259.08 227.33 0)
 		(unit 1)
