File: hardware/schematics/Laser Controllerv2_only_for_pcb_test.kicad_sch (KiCad schematic)
At the start: 122 parts, among them J1 SD Card Module (6-pin, 2.54mm), J2 12.6V IN (BUCK), J3 PWR IN Galvo, J4 FAN1 12V IN, J5 FAN1, J6 FAN2 12V IN, J7 FAN2, U1 ESP32-S3-N16R8-DevKit, U10 DS18B20 connector, U12 OPA4134UA_2K5, U13 Galvo Input, U15 6N137, U16 6N137, U17 6N137, U2 DAC8562SDGST, U3 TTL_RGB Blue, U4 TTL_RGB Red, U5 TTL_RGB Green, U6 DS18B20 connector, U7 DS18B20 connector, U8 DS18B20 connector, U9 DS18B20 connector

Commit message: fix(hw): specify SMD trigger diodes in v2.0.10
Match the existing SOD-123 pads to explicit manufacturer parts and reject recurring package warnings. Copper and connectivity stay unchanged.

Record user exclusion of further thermal, load and timing work; existing limitations remain unverified.
Parts:
- D_TRIGCL_SCAN1, D_TRIGCL_WD1: value 1N4148 -> 1N4148W; symbol Diode:1N4148 -> Diode:1N4148W; Assembly (none) -> SOD-123; cathode band to pad 1 (trigger); anode pad 2 to po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; MPN (none) -> 1N4148W-7-F; Manufacturer (none) -> Diodes Incorporated
Changed lines of the file:
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@@
 		(title "GalvOS ESP32 Laser Controller - V2 engineering review")
 		(date "2026-09-14")
-		(rev "V2.0.9 DRAFT - NOT FOR FABRICATION")
+		(rev "V2.0.10 DRAFT - NOT FOR FABRICATION")
 	)
 	(rectangle
@@
 (text "3V3 DMX input protection; no galvanic isolation" (at 187.96 346.71 0) (effects (font (size 1.27 1.27)) (justify left)))
 	(symbol
-		(lib_id "Diode:1N4148")
+		(lib_id "Diode:1N4148W")
 		(at 490.22 270.51 0)
 		(unit 1)
@@
 			)
 		)
-		(property "Value" "1N4148"
+		(property "Value" "1N4148W"
 			(at 490.22 266.70000000000005 0)
 			(show_name no)
@@
 			)
 		)
-		(property "Datasheet" "https://assets.nexperia.com/documents/data-sheet/1N4148_1N4448.pdf"
+		(property "Datasheet" "https://www.diodes.com/assets/Datasheets/ds30086.pdf"
 			(at 490.22 270.51 0)
 			(hide yes)
@@
 			)
 		)
-		(property "Description" "100V 0.15A standard switching diode, DO-35"
+		(property "Description" "100V 300mA fast switching diode, SOD-123; ratings subject to datasheet conditions"
 			(at 490.22 270.51 0)
 			(hide yes)
@@
 			)
 		)
+		(property "Manufacturer" "Diodes Incorporated"
+			(at 490.22 270.51 0)
+			(hide yes)
+			(effects (font (size 1.27 1.27)))
+		)
+		(property "MPN" "1N4148W-7-F"
+			(at 490.22 270.51 0)
+			(hide yes)
+			(effects (font (size 1.27 1.27)))
+		)
+		(property "Assembly" "SOD-123; cathode band to pad 1 (trigger); anode pad 2 to power ground. Negative clamp only, not complete timer-input protection."
+			(at 490.22 270.51 0)
+			(hide yes)
+			(effects (font (size 1.27 1.27)))
+		)
 		(pin "1"
 		)
@@
 	)
 	(symbol
-		(lib_id "Diode:1N4148")
+		(lib_id "Diode:1N4148W")
 		(at 490.22 355.6 0)
 		(unit 1)
@@
 			)
 		)
-		(property "Value" "1N4148"
+		(property "Value" "1N4148W"
 			(at 490.22 351.79 0)
 			(show_name no)
@@
 			)
 		)
-		(property "Datasheet" "https://assets.nexperia.com/documents/data-sheet/1N4148_1N4448.pdf"
+		(property "Datasheet" "https://www.diodes.com/assets/Datasheets/ds30086.pdf"
 			(at 490.22 355.6 0)
 			(hide yes)
@@
 			)
 		)
-		(property "Description" "100V 0.15A standard switching diode, DO-35"
+		(property "Description" "100V 300mA fast switching diode, SOD-123; ratings subject to datasheet conditions"
 			(at 490.22 355.6 0)
 			(hide yes)
@@
 			)
 		)
+		(property "Manufacturer" "Diodes Incorporated"
+			(at 490.22 355.6 0)
+			(hide yes)
+			(effects (font (size 1.27 1.27)))
+		)
+		(property "MPN" "1N4148W-7-F"
+			(at 490.22 355.6 0)
+			(hide yes)
+			(effects (font (size 1.27 1.27)))
+		)
+		(property "Assembly" "SOD-123; cathode band to pad 1 (trigger); anode pad 2 to power ground. Negative clamp only, not complete timer-input protection."
+			(at 490.22 355.6 0)
+			(hide yes)
+			(effects (font (size 1.27 1.27)))
+		)
 		(pin "1"
