File: hardware/snapshots/2026-09-15-visible-wires/Laser Controllerv2_only_for_pcb_test.kicad_sch (KiCad schematic)
At the start: 122 parts, among them J1 SD Card Module (6-pin, 2.54mm), J2 12.6V IN (BUCK), J3 PWR IN Galvo, J4 FAN1 12V IN, J5 FAN1, J6 FAN2 12V IN, J7 FAN2, U1 ESP32-S3-N16R8-DevKit, U10 DS18B20 connector, U12 OPA4134UA_2K5, U13 Galvo Input, U15 6N137, U16 6N137, U17 6N137, U2 DAC8562SDGST, U3 TTL_RGB Blue, U4 TTL_RGB Red, U5 TTL_RGB Green, U6 DS18B20 connector, U7 DS18B20 connector, U8 DS18B20 connector, U9 DS18B20 connector

Commit message: feat(hw): add visible-wire schematic copy
Connections:
- net Net-(C3-Pad1): no longer names the net of C3.1, R11.1, X_NODE1.1
- net Net-(C4-Pad1): no longer names the net of C4.1, R13.1, Y_NODE1.1
- net Net-(C_SCANX1-Pad2): no longer names the net of C_SCANX1.2, R7.2, X_NODE1.2
- net Net-(C_SCANY1-Pad2): no longer names the net of C_SCANY1.2, R14.2, Y_NODE1.2
- net Net-(U1-GPIO18): no longer names the net of R5.1, U1.J1_11 (GPIO18), U10.2 (Pin_2), U6.2 (Pin_2), U7.2 (Pin_2), U8.2 (Pin_2), U9.2 (Pin_2)
- net Net-(U12-+IN_A): no longer names the net of R10.1, R9.1, U12.3 (+IN_A)
- net Net-(U12-+IN_B): no longer names the net of R15.1, R25.1, U12.5 (+IN_B)
- net Net-(U12-+IN_C): no longer names the net of C2.1, U12.10 (+IN_C), U2.10 (VREFINNREFOUT)
- net Net-(U12--IN_A): no longer names the net of R12.2, R7.1, U12.2 (-IN_A)
- net Net-(U12--IN_B): no longer names the net of R14.1, R17.1, U12.6 (-IN_B)
- net Net-(U12--IN_D): no longer names the net of U12.13 (-IN_D), U12.14 (OUT_D)
- net Net-(U12-OUT_A): no longer names the net of R12.1, R6.1, U12.1 (OUT_A)
- net Net-(U12-OUT_B): no longer names the net of R16.1, R17.2, U12.7 (OUT_B)
- net Net-(U13-Pin_2): no longer names the net of R6.2, U13.2 (Pin_2)
- net Net-(U13-Pin_3): no longer names the net of R16.2, U13.3 (Pin_3)
- net Net-(U15-A): no longer names the net of R1.2, U15.2 (A)
- net Net-(U16-A): no longer names the net of R2.2, U16.2 (A)
- net Net-(U17-A): no longer names the net of R4.2, U17.2 (A)
- net Net-(U2-VOUTA): no longer names the net of R11.2, U2.1 (VOUTA)
- net Net-(U2-VOUTB): no longer names the net of R13.2, U2.2 (VOUTB)
- net Net-(U_DACLV1-B1): no longer names the net of R_DACSCLK1.2, U_DACLV1.21 (B1)
- net Net-(U_DACLV1-B2): no longer names the net of R_DACDIN1.2, U_DACLV1.20 (B2)
- net Net-(U_DACLV1-B3): no longer names the net of R_DACSYNC1.2, U_DACLV1.19 (B3)
- net Net-(U_DACLV1-B4): no longer names the net of R_DACCLR1.2, U_DACLV1.18 (B4)
Other:
- moved on the sheet: C1, C2, C3, C4, C5, C6, C7, C8, C9, C_ANA1, C_ANA2, C_BOOT1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
